File: eagle/BLDC Driver 4 Layer/BLDC driver board 4 layer.sch (EAGLE design)
At the start: 43 parts, among them Q1 CSD173XXQX-NEXFET, Q11 CSD173XXQX-NEXFET, Q3 CSD173XXQX-NEXFET, Q5 CSD173XXQX-NEXFET, Q7 CSD173XXQX-NEXFET, Q9 CSD173XXQX-NEXFET

Commit message: More changes to bldc 4-layer, cleaned up files.
Parts:
- removed R4, R5, R6: 1k, CMPE118lib:RESISTOR1206
- removed U$1: CAN_NODE_SHIELD_V3, ASL:CAN_NODE_SHIELD_V3
- added RN1: (no value), ASL:RESISTOR_ARRAY-4
- added U$2: CAN_NODE_SHIELD_V3, ASL:CAN_NODE_SHIELD_V3
Connections:
- net 3V3: now also U$2.VCC3V3@10, U$2.VCC3V3@24; no longer U$1.CAN_HI, U$1.RB14
- net ADC/HALL1: now also RN1.2, U$2.RB0; no longer R6.1, U$1.RB1
- net ADC/HALL2: now also RN1.3, U$2.RB1; no longer R5.1, U$1.RB2
- net ADC/HALL3: now also RN1.1, U$2.RB2; no longer R4.1, U$1.VCC3V3@10
- net CRRNTSNS1: now also U$2.RA2; no longer U$1.RB8
- net CRRNTSNS2: now also U$2.RA0; no longer U$1.MCLR
- net GND: now also U$2.GND@1, U$2.GND@13, U$2.GND@14, U$2.GND@15, U$2.GND@16, U$2.GND@2, U$2.GND@27, U$2.GND@28; no longer U$1.GND@14, U$1.GND@16, U$1.GND@2, U$1.GND@28, U$1.PGD, U$1.RB12
- net N$13: now also RN1.6, RN1.7, RN1.8; no longer R4.2, R5.2, R6.2
- net PWM1: now also U$2.RB8; no longer U$1.PGC
- net PWM2: now also U$2.RB12; no longer U$1.RB9
- net PWM3: now also U$2.RB14; no longer U$1.RB15
- net QEI-A: now also U$2.RB10; no longer U$1.VCC5V0@20
- net QEI-B: now also U$2.RB9; no longer U$1.RB10
- net QEI-INDEX: now also U$2.RB15; no longer U$1.GND@13
- net VCC: now also U$2.VCC5V0@20, U$2.VCC5V0@6; no longer U$1.RA2, U$1.RB0
Other:
- moved on the sheet: JP3

Commit message: 4-layer bldc work, finding more space.
Parts:
- removed 5V: (no value), jumper:JP1E
- removed ADC/HALL, QEI: (no value), CMPE118lib:M03LOCK_NO_SILK
- removed LED3: (no value), ASL:LED1206
- removed R18: 330, ASL:RESISTOR0805-RES
- added J1: (no value), ASL:M02
- added JP1: (no value), ASL:M06SMD-STRAIGHT
Connections:
- removed net N$11: DRV8301.PWRGD, R18.1
- removed net N$15: LED3.C, R18.2
- new net N$2: DRV8301.FAULT', U$2.PGC
- net 3V3: no longer LED3.A
- net ADC/HALL1: now also JP1.6; no longer ADC/HALL.3
- net ADC/HALL2: now also JP1.5; no longer ADC/HALL.2
- net ADC/HALL3: now also JP1.4; no longer ADC/HALL.1
- net GND: now also J1.1; no longer 5V.1
- net QEI-A: now also JP1.3; no longer QEI.3
- net QEI-B: now also JP1.2; no longer QEI.2
- net QEI-INDEX: now also JP1.1; no longer QEI.1
- net VCC: now also J1.2; no longer 5V.2
Changed lines of the file:
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@@
 <part name="P+6" library="CMPE118lib" deviceset="VCC" device=""/>
 <part name="VIN" library="CMPE118lib" deviceset="SCREWTERM02" device="" value=""/>
-<part name="QEI" library="CMPE118lib" deviceset="M03" device="LOCK_NO_SILK"/>
-<part name="ADC/HALL" library="CMPE118lib" deviceset="M03" device="LOCK_NO_SILK"/>
-<part name="5V" library="jumper" deviceset="JP1E" device=""/>
 <part name="DRV8301" library="ASL" deviceset="DRV8302" device=""/>
 <part name="R2" library="ASL" deviceset="RESISTOR" device="0805-RES" value="1M"/>
@@
 <part name="R12" library="ASL" deviceset="RESISTOR" device="0805-RES" value="3.16k"/>
 <part name="R11" library="ASL" deviceset="RESISTOR" device="0805-RES" value="10k"/>
-<part name="LED3" library="ASL" deviceset="LED" device="1206"/>
-<part name="R18" library="ASL" deviceset="RESISTOR" device="0805-RES" value="330"/>
 <part name="Q1" library="ASL" deviceset="CSD173XXQX" device="-NEXFET"/>
 <part name="Q3" library="ASL" deviceset="CSD173XXQX" device="-NEXFET"/>
@@
 <part name="RN1" library="ASL" deviceset="RESISTOR_ARRAY-4" device=""/>
 <part name="U$2" library="ASL" deviceset="CAN_NODE_SHIELD_V3" device=""/>
+<part name="JP1" library="ASL" deviceset="M06" device="SMD-STRAIGHT"/>
+<part name="J1" library="ASL" deviceset="M02" device=""/>
 </parts>
 <sheets>
@@
 <instance part="P+6" gate="1" x="63.5" y="137.16"/>
 <instance part="VIN" gate="G$1" x="35.56" y="137.16" rot="R270"/>
-<instance part="QEI" gate="G$1" x="30.48" y="83.82"/>
-<instance part="ADC/HALL" gate="G$1" x="30.48" y="63.5"/>
-<instance part="5V" gate="A" x="119.38" y="127" rot="R90"/>
 <instance part="DRV8301" gate="U1" x="43.18" y="-53.34"/>
 <instance part="R2" gate="G$1" x="83.82" y="-43.18" rot="MR270"/>
@@
 <instance part="R12" gate="G$1" x="-27.94" y="-63.5" rot="MR270"/>
 <instance part="R11" gate="G$1" x="-27.94" y="-73.66" rot="MR270"/>
-<instance part="LED3" gate="G$1" x="0" y="-22.86" rot="MR270"/>
-<instance part="R18" gate="G$1" x="12.7" y="-22.86" rot="R180"/>
 <instance part="Q1" gate="G$1" x="172.72" y="-45.72"/>
 <instance part="Q3" gate="G$1" x="172.72" y="-93.98"/>
@@
 <instance part="RN1" gate="G$1" x="66.04" y="127" rot="R90"/>
 <instance part="U$2" gate="G$1" x="45.72" y="25.4"/>
+<instance part="JP1" gate="G$1" x="33.02" y="78.74"/>
+<instance part="J1" gate="G$1" x="111.76" y="124.46"/>
 </instances>
 <busses>
@@
 </segment>
 <segment>
-<pinref part="5V" gate="A" pin="2"/>
 <wire x1="121.92" y1="129.54" x2="129.54" y2="129.54" width="0.2032" layer="91"/>
 <label x="129.54" y="129.54" size="1.778" layer="95"/>
+<pinref part="J1" gate="G$1" pin="2"/>
+<junction x="121.92" y="129.54"/>
 </segment>
 <segment>
@@
 <net name="GND" class="0">
 <segment>
-<pinref part="5V" gate="A" pin="1"/>
 <wire x1="121.92" y1="127" x2="129.54" y2="127" width="0.2032" layer="91"/>
 <label x="129.54" y="127" size="1.778" layer="95"/>
+<pinref part="J1" gate="G$1" pin="1"/>
+<junction x="121.92" y="127"/>
 </segment>
 <segment>
@@
 </segment>
 <segment>
-<wire x1="38.1" y1="60.96" x2="40.64" y2="60.96" width="0.2032" layer="91"/>
-<label x="40.64" y="60.96" size="1.778" layer="95"/>
-<pinref part="ADC/HALL" gate="G$1" pin="3"/>
+<wire x1="38.1" y1="73.66" x2="40.64" y2="73.66" width="0.2032" layer="91"/>
+<label x="40.64" y="73.66" size="1.778" layer="95"/>
+<pinref part="JP1" gate="G$1" pin="6"/>
+<junction x="38.1" y="73.66"/>
 </segment>
 <segment>
@@
 </segment>
 <segment>
-<wire x1="38.1" y1="63.5" x2="40.64" y2="63.5" width="0.2032" layer="91"/>
-<label x="40.64" y="63.5" size="1.778" layer="95"/>
-<pinref part="ADC/HALL" gate="G$1" pin="2"/>
+<wire x1="38.1" y1="76.2" x2="40.64" y2="76.2" width="0.2032" layer="91"/>
+<label x="40.64" y="76.2" size="1.778" layer="95"/>
+<pinref part="JP1" gate="G$1" pin="5"/>
+<junction x="38.1" y="76.2"/>
 </segment>
 <segment>
@@
 </segment>
 <segment>
-<wire x1="38.1" y1="66.04" x2="40.64" y2="66.04" width="0.2032" layer="91"/>
-<label x="40.64" y="66.04" size="1.778" layer="95"/>
-<pinref part="ADC/HALL" gate="G$1" pin="1"/>
+<wire x1="38.1" y1="78.74" x2="40.64" y2="78.74" width="0.2032" layer="91"/>
+<label x="40.64" y="78.74" size="1.778" layer="95"/>
+<pinref part="JP1" gate="G$1" pin="4"/>
+<junction x="38.1" y="78.74"/>
 </segment>
 <segment>
@@
 <wire x1="38.1" y1="83.82" x2="40.64" y2="83.82" width="0.2032" layer="91"/>
 <label x="40.64" y="83.82" size="1.778" layer="95"/>
-<pinref part="QEI" gate="G$1" pin="2"/>
+<pinref part="JP1" gate="G$1" pin="2"/>
+<junction x="38.1" y="83.82"/>
 </segment>
 </net>
@@
 <wire x1="38.1" y1="81.28" x2="40.64" y2="81.28" width="0.2032" layer="91"/>
 <label x="40.64" y="81.28" size="1.778" layer="95"/>
-<pinref part="QEI" gate="G$1" pin="3"/>
+<pinref part="JP1" gate="G$1" pin="3"/>
+<junction x="38.1" y="81.28"/>
 </segment>
 </net>
@@
 <wire x1="38.1" y1="86.36" x2="40.64" y2="86.36" width="0.2032" layer="91"/>
 <label x="40.64" y="86.36" size="1.778" layer="95"/>
-<pinref part="QEI" gate="G$1" pin="1"/>
+<pinref part="JP1" gate="G$1" pin="1"/>
+<junction x="38.1" y="86.36"/>
 </segment>
 </net>
@@
 <wire x1="25.4" y1="-38.1" x2="22.86" y2="-38.1" width="0.2032" layer="91"/>
 <label x="17.78" y="-38.1" size="1.778" layer="95"/>
-</segment>
-<segment>
-<label x="-5.08" y="-5.08" size="1.778" layer="95"/>
-<wire x1="-5.08" y1="-5.08" x2="-5.08" y2="-22.86" width="0.2032" layer="91"/>
-<pinref part="LED3" gate="G$1" pin="A"/>
-<wire x1="-5.08" y1="-22.86" x2="-2.54" y2="-22.86" width="0.2032" layer="91"/>
 </segment>
 <segment>
@@
 </segment>
 </net>
-<net name="N$15" class="0">
-<segment>
-<pinref part="LED3" gate="G$1" pin="C"/>
-<pinref part="R18" gate="G$1" pin="2"/>
-<wire x1="5.08" y1="-22.86" x2="7.62" y2="-22.86" width="0.1524" layer="91"/>
-</segment>
-</net>
 <net name="N$13" class="0">
 <segment>
@@
 </segment>
 </net>
-<net name="N$11" class="0">
-<segment>
-<pinref part="R18" gate="G$1" pin="1"/>
-<wire x1="17.78" y1="-22.86" x2="20.32" y2="-22.86" width="0.2032" layer="91"/>
-<wire x1="20.32" y1="-22.86" x2="20.32" y2="-27.94" width="0.2032" layer="91"/>
-<pinref part="DRV8301" gate="U1" pin="PWRGD"/>
-<wire x1="20.32" y1="-27.94" x2="25.4" y2="-27.94" width="0.2032" layer="91"/>
-</segment>
-</net>
+<net name="N$2" class="0">
+<segment>
+<pinref part="U$2" gate="G$1" pin="PGC"/>
+<wire x1="22.86" y1="27.94" x2="0" y2="27.94" width="0.2032" layer="91"/>
+<wire x1="0" y1="27.94" x2="0" y2="-33.02" width="0.2032" layer="91"/>
+<pinref part="DRV8301" gate="U1" pin="FAULT'"/>
+<wire x1="0" y1="-33.02" x2="25.4" y2="-33.02" width="0.2032" layer="91"/>
+</segment>
+</net>

Commit message: Updated some footprints.
Parts:
- DRV8301: device ASL:DRV8302 -> pavlo:DRV8302
Other:
- moved on the sheet: DRV8301
Changed lines of the file:
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@@
 <part name="P+6" library="CMPE118lib" deviceset="VCC" device=""/>
 <part name="VIN" library="CMPE118lib" deviceset="SCREWTERM02" device="" value=""/>
-<part name="DRV8301" library="ASL" deviceset="DRV8302" device=""/>
+<part name="DRV8301" library="pavlo" deviceset="DRV8302" device=""/>
 <part name="R2" library="ASL" deviceset="RESISTOR" device="0805-RES" value="1M"/>
 <part name="C1" library="ASL" deviceset="CAP" device="1206" value=".015uF"/>
@@
 <pinref part="DRV8301" gate="U1" pin="EN_GATE"/>
 <wire x1="25.4" y1="-58.42" x2="20.32" y2="-58.42" width="0.2032" layer="91"/>
-</segment>
-</net>
+<label x="15.24" y="-58.42" size="1.778" layer="95"/>
+</segment>
+</net>

Commit message: exploded 4-layer bldc due to space boon
Parts:
- removed DRV8301: DRV8302, pavlo:DRV8302
- removed Q11, Q7, Q9: CSD173XXQX-NEXFET, ASL:CSD173XXQX-NEXFET
- removed R7: .01, ASL:RESISTOR
- added Q2, Q4, Q6: CSD173XXQX-NEXFET, pavlo:CSD173XXQX-NEXFET
- added R4: .01, pavlo:RESISTOR
- added U$1: DRV8302-56, pavlo:DRV8302-56
- C6: device ASL:CAP_POLE -> pavlo:CAP_POL
- C7: device ASL:CAP_POLE -> pavlo:CAP_POLYO
- Q1, Q3, Q5: device ASL:CSD173XXQX-NEXFET -> pavlo:CSD173XXQX-NEXFET
- R3: device ASL:RESISTOR -> pavlo:RESISTOR
Connections:
- net 3V3: now also U$1.EN_GATE, U$1.M_PWM, U$1.REF; no longer DRV8301.EN_GATE, DRV8301.M_PWM, DRV8301.REF
- net CRRNTSNS1: now also U$1.SO1; no longer DRV8301.SO1
- net CRRNTSNS2: now also U$1.SO2; no longer DRV8301.SO2
- net GH_A: now also Q1.G, U$1.GH_A; no longer DRV8301.GH_A, Q11.G
- net GH_B: now also Q3.G, U$1.GH_B; no longer DRV8301.GH_B, Q1.G
- net GH_C: now also Q5.G, U$1.GH_C; no longer DRV8301.GH_C, Q3.G
- net GL_A: now also Q2.G, U$1.GL_A; no longer DRV8301.GL_A, Q9.G
- net GL_B: now also Q4.G, U$1.GL_B; no longer DRV8301.GL_B, Q7.G
- net GL_C: now also Q6.G, U$1.GL_C; no longer DRV8301.GL_C, Q5.G
- net GND: now also U$1.AGND, U$1.DC_CAL, U$1.DTC, U$1.GAIN, U$1.GND, U$1.M_OC; no longer DRV8301.AGND, DRV8301.DC_CAL, DRV8301.DTC, DRV8301.GAIN, DRV8301.GND, DRV8301.M_OC
- net N$1: now also U$1.SS_TR; no longer DRV8301.SS_TR
- net N$10: now also U$1.EN_BUCK; no longer DRV8301.EN_BUCK
- net N$12: now also U$1.OC_ADJ; no longer DRV8301.OC_ADJ
- net N$16: now also U$1.AVDD; no longer DRV8301.AVDD
- net N$18: now also U$1.DVDD; no longer DRV8301.DVDD
- net N$19: now also U$1.CP1; no longer DRV8301.CP1
- net N$2: now also U$1.FAULT'; no longer DRV8301.FAULT'
- net N$20: now also U$1.CP2; no longer DRV8301.CP2
- net N$21: now also U$1.GVDD; no longer DRV8301.GVDD
- net N$3: now also U$1.BIAS; no longer DRV8301.BIAS
- net N$4: now also U$1.BST_A; no longer DRV8301.BST_A
- net N$6: now also U$1.BST_B; no longer DRV8301.BST_B
- net N$8: now also U$1.BST_C; no longer DRV8301.BST_C
- net OUTPUTA: now also Q1.S, Q2.D, U$1.SH_A; no longer DRV8301.SH_A, Q11.S, Q9.D
- net OUTPUTB: now also Q3.S, Q4.D, U$1.SH_B; no longer DRV8301.SH_B, Q1.S, Q7.D
- net OUTPUTC: now also Q5.S, Q6.D, U$1.SH_C; no longer DRV8301.SH_C, Q3.S, Q5.D
- net PWM1: now also U$1.INH_A; no longer DRV8301.INH_A
- net PWM2: now also U$1.INH_B; no longer DRV8301.INH_B
- net PWM3: now also U$1.INH_C; no longer DRV8301.INH_C
- net SN1: now also Q4.S, R4.1, U$1.SL_B, U$1.SN1; no longer DRV8301.SL_B, DRV8301.SN1, Q7.S, R7.2
- net SN2: now also Q2.S, R3.1, U$1.SL_A, U$1.SN2; no longer DRV8301.SL_A, DRV8301.SN2, Q9.S, R3.2
- net VNEG: now also Q6.S, R3.2, R4.2, U$1.SL_C, U$1.SP1, U$1.SP2; no longer DRV8301.SL_C, DRV8301.SP1, DRV8301.SP2, Q5.S, R3.1, R7.1
- net V_BATT: now also Q5.D, U$1.PVDD1, U$1.PVDD2, U$1.PVDD2(1); no longer DRV8301.PVDD1, DRV8301.PVDD2, DRV8301.PVDD2(1), Q11.D
Other:
- moved on the sheet: C6, C7, Q1, Q3, Q5, R3

Commit message: Completed BLDC 4-layer and new Ether-shield
Parts:
- removed OUTPUT: (no value), con-wago-500:W237-103
- removed RN1: (no value), ASL:RESISTOR_ARRAY-4
- added JP2: M03PTH, ASL:M03PTH
- added JP4: M03-SCREW-5MM, ASL:M03-SCREW-5MM
- added R5, R6, R7: (no value), ASL:RESISTOR0805-RES
- JP1: value (none) -> M03PTH; device ASL:M06SMD-STRAIGHT -> ASL:M03PTH
- U$2: value CAN_NODE_SHIELD_V3 -> CANODE_SHIELD; device ASL:CAN_NODE_SHIELD_V3 -> ASL:CANODE_SHIELD
Connections:
- net ADC/HALL1: now also JP2.3, R6.1; no longer JP1.6, RN1.2
- net ADC/HALL2: now also JP2.2, R7.1; no longer JP1.5, RN1.3
- net ADC/HALL3: now also JP2.1, R5.1; no longer JP1.4, RN1.1
- net N$13: now also R5.2, R6.2, R7.2; no longer RN1.6, RN1.7, RN1.8
- net OUTPUTA: now also JP4.1; no longer OUTPUT-1.KL
- net OUTPUTB: now also JP4.2; no longer OUTPUT-2.KL
- net OUTPUTC: now also JP4.3; no longer OUTPUT-3.KL

Commit message: Ready for Board Run.
Parts:
- added R9: 3.3k, ASL:RESISTOR0805-RES
Connections:
- net 3V3: now also R9.1
- net N$2: now also R9.2
Changed lines of the file:
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@@
 <?xml version="1.0" encoding="utf-8"?>
 <!DOCTYPE eagle SYSTEM "eagle.dtd">
-<eagle version="6.4">
+<eagle version="6.1">
 <drawing>
 <settings>
@@
 <part name="R6" library="ASL" deviceset="RESISTOR" device="0805-RES"/>
 <part name="R7" library="ASL" deviceset="RESISTOR" device="0805-RES"/>
+<part name="R9" library="ASL" deviceset="RESISTOR" device="0805-RES" value="3.3k"/>
 </parts>
 <sheets>
@@
 <instance part="R6" gate="G$1" x="66.04" y="129.54" rot="R90"/>
 <instance part="R7" gate="G$1" x="68.58" y="129.54" rot="R90"/>
+<instance part="R9" gate="G$1" x="-5.08" y="-17.78"/>
 </instances>
 <busses>
@@
 <label x="15.24" y="-58.42" size="1.778" layer="95"/>
 <pinref part="U$1" gate="U1" pin="EN_GATE"/>
+</segment>
+<segment>
+<pinref part="R9" gate="G$1" pin="1"/>
+<wire x1="-10.16" y1="-17.78" x2="-27.94" y2="-17.78" width="0.1524" layer="91"/>
+<wire x1="-27.94" y1="-17.78" x2="-27.94" y2="-15.24" width="0.1524" layer="91"/>
+<label x="-27.94" y="-15.24" size="1.778" layer="95"/>
 </segment>
 </net>
@@
 <pinref part="U$2" gate="G$1" pin="PGC"/>
 <wire x1="22.86" y1="27.94" x2="0" y2="27.94" width="0.2032" layer="91"/>
-<wire x1="0" y1="27.94" x2="0" y2="-33.02" width="0.2032" layer="91"/>
+<wire x1="0" y1="27.94" x2="0" y2="-17.78" width="0.2032" layer="91"/>
+<wire x1="0" y1="-17.78" x2="0" y2="-33.02" width="0.2032" layer="91"/>
 <wire x1="0" y1="-33.02" x2="25.4" y2="-33.02" width="0.2032" layer="91"/>
 <pinref part="U$1" gate="U1" pin="FAULT'"/>
 <pinref part="U$2" gate="G$1" pin="PGC"/>
 <junction x="22.86" y="27.94"/>
-</segment>
-</net>
+<pinref part="R9" gate="G$1" pin="2"/>
+<junction x="0" y="-17.78"/>
+</segment>
+</net>
