File: eagle/MAC.PHY_shield/MAC.PHY_shield.brd (EAGLE design)
At the start: 49.9 x 49.9 mm, 25 parts, among them IC1 ENC28J60, Q1 CSM-7X-DU

Commit message: Polished up MAC-PHY Board.
Parts:
- removed E$1, E$2: (no value), ASL:STAND-OFF-TIGHT
- renumbered U$4 to F1
Other:
- board text added: "MAC/PHY Ethernet Shield"
- board text added: "v2.4"
Changed lines of the file:
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@@
 <?xml version="1.0" encoding="utf-8"?>
 <!DOCTYPE eagle SYSTEM "eagle.dtd">
-<eagle version="6.1">
+<eagle version="6.4">
 <drawing>
 <settings>
@@
 <setting verticaltext="up"/>
 </settings>
-<grid distance="0.01" unitdist="inch" unit="mm" style="lines" multiple="1" display="yes" altdistance="0.001" altunitdist="inch" altunit="mm"/>
+<grid distance="0.01" unitdist="mm" unit="mm" style="lines" multiple="1" display="yes" altdistance="0.005" altunitdist="mm" altunit="mm"/>
 <layers>
 <layer number="1" name="Top" color="4" fill="1" visible="yes" active="yes"/>
@@
 <layer number="49" name="Reference" color="7" fill="1" visible="no" active="yes"/>
 <layer number="50" name="dxf" color="7" fill="1" visible="no" active="no"/>
-<layer number="51" name="tDocu" color="7" fill="1" visible="yes" active="yes"/>
-<layer number="52" name="bDocu" color="7" fill="1" visible="yes" active="yes"/>
+<layer number="51" name="tDocu" color="7" fill="1" visible="no" active="yes"/>
+<layer number="52" name="bDocu" color="7" fill="1" visible="no" active="yes"/>
 <layer number="53" name="tGND_GNDA" color="7" fill="9" visible="no" active="no"/>
 <layer number="54" name="bGND_GNDA" color="1" fill="9" visible="no" active="no"/>
@@
 <wire x1="13.843" y1="58.801" x2="10.16" y2="55.118" width="0" layer="20" curve="90"/>
 <wire x1="10.16" y1="55.118" x2="10.16" y2="12.5984" width="0" layer="20"/>
+<text x="59.182" y="36.322" size="0.8128" layer="21" rot="R90">MAC/PHY Ethernet Shield</text>
+<text x="59.182" y="50.038" size="0.8128" layer="21" rot="R90">v2.4</text>
 </plain>
 <attributes>
@@
 </class>
 </classes>
-<designrules>
+<designrules name="default">
 <description language="de">&lt;b&gt;EAGLE Design Rules&lt;/b&gt;
 &lt;p&gt;
@@
 <attribute name="MF" value="" x="85.8774" y="3.0226" size="1.778" layer="27" display="off"/>
 <attribute name="OC_FARNELL" value="unknown" x="85.8774" y="3.0226" size="1.778" layer="27" display="off"/>
-<attribute name="NAME" x="23.7021" y="46.3865" size="0.6096" layer="25"/>
+<attribute name="NAME" x="27.2581" y="47.6565" size="1.4224" layer="25"/>
 </element>
 <element name="U$1" library="ASL" package="CANODE_SHIELD" value="CANODE_SHIELD" x="10.16" y="8.89" smashed="yes"/>
 <element name="IC1" library="ASL" package="SOIC28-W" value="ENC28J60" x="24.638" y="31.7754" smashed="yes" rot="R180">
-<attribute name="NAME" x="25.8725" y="35.1229" size="0.6096" layer="25" ratio="15" rot="R180"/>
-<attribute name="VALUE" x="28.73" y="11.9454" size="1.27" layer="27" ratio="15" rot="R180"/>
-</element>
-<element name="U$3" library="ASL" package="08B0-1X1T-06-F" value="MAGJACK" x="35.052" y="36.068"/>
+<attribute name="NAME" x="25.8725" y="35.1229" size="1.4224" layer="25" ratio="15" rot="R180"/>
+<attribute name="VALUE" x="28.73" y="11.9454" size="1.4224" layer="27" ratio="15" rot="R180"/>
+</element>
+<element name="U$3" library="ASL" package="08B0-1X1T-06-F" value="MAGJACK" x="35.052" y="36.068" smashed="yes"/>
 <element name="C2" library="ASL" package="1206" value="10uF" x="32.0675" y="23.7744" smashed="yes" rot="R90">
-<attribute name="NAME" x="34.163" y="23.2029" size="0.6096" layer="25" ratio="10" rot="R90"/>
+<attribute name="NAME" x="34.671" y="22.6949" size="1.4224" layer="25" ratio="10" rot="R90"/>
 </element>
 <element name="R2" library="ASL" package="0805" value="300" x="26.0604" y="19.2913" smashed="yes" rot="R180">
-<attribute name="NAME" x="24.8539" y="21.5773" size="0.6096" layer="25" ratio="15" rot="R180"/>
+<attribute name="NAME" x="24.8539" y="21.5773" size="1.4224" layer="25" ratio="15" rot="R180"/>
 </element>
 <element name="R3" library="ASL" package="0805" value="300" x="55.3085" y="43.18" smashed="yes">
-<attribute name="NAME" x="56.007" y="42.2275" size="0.6096" layer="25" ratio="15" rot="R270"/>
+<attribute name="NAME" x="56.4515" y="45.593" size="1.4224" layer="25" ratio="15" rot="R180"/>
 </element>
 <element name="R4" library="ASL" package="0805" value="49.9" x="43.2054" y="27.4066" smashed="yes" rot="R90">
-<attribute name="NAME" x="41.9354" y="26.9621" size="0.6096" layer="25" ratio="15" rot="R90"/>
+<attribute name="NAME" x="42.4434" y="26.2001" size="1.4224" layer="25" ratio="15" rot="R90"/>
 </element>
 <element name="R5" library="ASL" package="0805" value="49.9" x="43.2308" y="21.717" smashed="yes" rot="R270">
-<attribute name="NAME" x="41.3258" y="22.225" size="0.6096" layer="25" ratio="15" rot="R270"/>
+<attribute name="NAME" x="41.3258" y="22.225" size="1.4224" layer="25" ratio="15" rot="R270"/>
 </element>
 <element name="R6" library="ASL" package="0805" value="49.9" x="37.8206" y="21.7805" smashed="yes" rot="R90">
-<attribute name="NAME" x="36.6776" y="21.844" size="0.6096" layer="25" ratio="15" rot="R90"/>
+<attribute name="NAME" x="38.862" y="20.1676" size="1.4224" layer="25" ratio="15" rot="R180"/>
 </element>
 <element name="R7" library="ASL" package="0805" value="49.9" x="37.8079" y="27.4193" smashed="yes" rot="R270">
-<attribute name="NAME" x="37.9984" y="24.7523" size="0.6096" layer="25" ratio="15" rot="R90"/>
-</element>
-<element name="U$4" library="ASL" package="1206" value="FERRITE_BEAD" x="47.9044" y="23.2029" smashed="yes" rot="R180">
-<attribute name="NAME" x="48.7299" y="21.8694" size="0.6096" layer="25" ratio="10" rot="R180"/>
-<attribute name="VALUE" x="49.8729" y="25.0444" size="0.4064" layer="27" rot="R180"/>
+<attribute name="NAME" x="36.9824" y="26.2763" size="1.4224" layer="25" ratio="15" rot="R90"/>
+</element>
+<element name="F1" library="ASL" package="1206" value="FERRITE_BEAD" x="47.9044" y="23.2029" smashed="yes" rot="R180">
+<attribute name="NAME" x="48.7299" y="21.8694" size="1.4224" layer="25" ratio="10" rot="R180"/>
 </element>
 <element name="C3" library="ASL" package="1206" value=".1 uF" x="47.8917" y="26.4033" smashed="yes">
-<attribute name="NAME" x="47.0027" y="27.8638" size="0.6096" layer="25" ratio="10"/>
+<attribute name="NAME" x="47.0027" y="27.8638" size="1.4224" layer="25" ratio="10"/>
 </element>
 <element name="C4" library="ASL" package="1206" value=".1 uF" x="40.5511" y="31.0769" smashed="yes">
-<attribute name="NAME" x="37.1475" y="26.8224" size="0.6096" layer="25" ratio="10"/>
+<attribute name="NAME" x="40.1955" y="32.1564" size="1.4224" layer="25" ratio="10"/>
 </element>
 <element name="R8" library="ASL" package="0805" value="2.32 k" x="35.0647" y="32.8295" smashed="yes" rot="R270">
-<attribute name="NAME" x="36.1442" y="34.544" size="0.6096" layer="25" ratio="15" rot="R270"/>
+<attribute name="NAME" x="33.9598" y="31.496" size="1.4224" layer="25" ratio="15" rot="R90"/>
 </element>
 <element name="C5" library="ASL" package="1206" value="33 pF" x="13.1191" y="45.3263" smashed="yes" rot="R180">
-<attribute name="NAME" x="13.5001" y="43.8023" size="0.6096" layer="25" ratio="10" rot="R180"/>
+<attribute name="NAME" x="14.0081" y="48.3743" size="1.4224" layer="25" ratio="10" rot="R180"/>
 </element>
 <element name="C6" library="ASL" package="1206" value="33 pF" x="13.1191" y="42.7736" smashed="yes" rot="R180">
-<attribute name="NAME" x="13.7541" y="41.3766" size="0.6096" layer="25" ratio="10" rot="R180"/>
+<attribute name="NAME" x="18.3261" y="43.4086" size="1.4224" layer="25" ratio="10" rot="R180"/>
 </element>
 <element name="C7" library="ASL" package="1206" value=".1 uF" x="49.4792" y="31.4198" smashed="yes" rot="R270">
-<attribute name="NAME" x="50.8762" y="31.8643" size="0.6096" layer="25" ratio="10" rot="R270"/>
+<attribute name="NAME" x="51.1302" y="31.8643" size="1.4224" layer="25" ratio="10" rot="R270"/>
 </element>
 <element name="C8" library="ASL" package="1206" value=".1 uF" x="13.1191" y="38.6207" smashed="yes">
-<attribute name="NAME" x="12.7381" y="39.8272" size="0.6096" layer="25" ratio="10"/>
+<attribute name="NAME" x="11.7221" y="36.0172" size="1.4224" layer="25" ratio="10"/>
 </element>
 <element name="C9" library="ASL" package="1206" value=".1 uF" x="55.4863" y="40.0177" smashed="yes" rot="R180">
-<attribute name="NAME" x="55.9943" y="41.9227" size="0.6096" layer="25" ratio="10" rot="R180"/>
+<attribute name="NAME" x="56.7563" y="38.6207" size="1.4224" layer="25" ratio="10" rot="R180"/>
 </element>
 <element name="C10" library="ASL" package="1206" value=".1 uF" x="20.3073" y="18.1991" smashed="yes">
-<attribute name="NAME" x="23.4188" y="17.8181" size="0.6096" layer="25" ratio="10"/>
-</element>
-<element name="E$1" library="ASL" package="STAND-OFF-TIGHT" value="" x="56.388" y="12.5984"/>
-<element name="E$2" library="ASL" package="STAND-OFF-TIGHT" value="" x="13.843" y="12.573"/>
-<element name="E$3" library="ASL" package="STAND-OFF-TIGHT" value="" x="13.843" y="55.118"/>
-<element name="E$4" library="ASL" package="STAND-OFF-TIGHT" value="" x="56.388" y="55.118"/>
+<attribute name="NAME" x="23.4188" y="17.8181" size="1.4224" layer="25" ratio="10"/>
+</element>
+<element name="E$3" library="ASL" package="STAND-OFF-TIGHT" value="" x="13.843" y="55.118" smashed="yes"/>
+<element name="E$4" library="ASL" package="STAND-OFF-TIGHT" value="" x="56.388" y="55.118" smashed="yes"/>
 </elements>
 <signals>
@@
 <via x="35.56" y="39.878" extent="1-16" drill="0.6"/>
 <via x="49.276" y="39.878" extent="1-16" drill="0.6"/>
-<wire x1="49.502" y1="36.068" x2="49.276" y2="39.878" width="0" layer="19" extent="1-1"/>
 <wire x1="29.238" y1="36.0754" x2="35.052" y2="36.068" width="0" layer="19" extent="1-16"/>
 </signal>
@@
 <contactref element="R5" pad="1"/>
 <contactref element="U$3" pad="1"/>
-<contactref element="U$4" pad="2"/>
+<contactref element="F1" pad="2"/>
 <contactref element="C3" pad="1"/>
 <wire x1="46.5044" y1="23.2029" x2="43.8167" y2="23.2029" width="0.3048" layer="1"/>
@@
 <contactref element="U$1" pad="3V3"/>
 <contactref element="U$1" pad="3V31"/>
-<contactref element="U$4" pad="1"/>
+<contactref element="F1" pad="1"/>
 <contactref element="IC1" pad="P$25"/>
 <contactref element="C7" pad="2"/>
@@
 </signal>
 </signals>
-<errors>
-</errors>
 </board>
 </drawing>

Commit message: Ready for Board Run.
Other:
- outline, holes or cut-outs redrawn
Changed lines of the file:
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@@
 <?xml version="1.0" encoding="utf-8"?>
 <!DOCTYPE eagle SYSTEM "eagle.dtd">
-<eagle version="6.4">
+<eagle version="6.1">
 <drawing>
 <settings>
@@
 <layer number="27" name="tValues" color="7" fill="1" visible="yes" active="yes"/>
 <layer number="28" name="bValues" color="7" fill="1" visible="yes" active="yes"/>
-<layer number="29" name="tStop" color="7" fill="3" visible="no" active="yes"/>
-<layer number="30" name="bStop" color="7" fill="6" visible="no" active="yes"/>
+<layer number="29" name="tStop" color="7" fill="3" visible="yes" active="yes"/>
+<layer number="30" name="bStop" color="7" fill="6" visible="yes" active="yes"/>
 <layer number="31" name="tCream" color="7" fill="4" visible="no" active="yes"/>
 <layer number="32" name="bCream" color="7" fill="5" visible="no" active="yes"/>
@@
 <board>
 <plain>
-<wire x1="10.16" y1="12.5984" x2="13.8684" y2="8.89" width="0" layer="20" curve="90"/>
 <wire x1="13.8684" y1="8.89" x2="13.8938" y2="8.89" width="0" layer="20"/>
-<wire x1="13.8938" y1="8.89" x2="17.5514" y2="12.5476" width="0" layer="20" curve="90"/>
-<wire x1="17.5514" y1="12.5476" x2="17.5514" y2="15.3924" width="0" layer="20"/>
-<wire x1="17.5514" y1="15.3924" x2="18.1356" y2="15.7226" width="0" layer="20" curve="-90"/>
 <wire x1="18.1356" y1="15.7226" x2="35.0774" y2="15.7226" width="0" layer="20"/>
 <wire x1="35.0774" y1="15.7226" x2="35.5854" y2="15.4686" width="0" layer="20" curve="-90"/>
@@
 <wire x1="56.388" y1="58.801" x2="13.843" y2="58.801" width="0" layer="20"/>
 <wire x1="13.843" y1="58.801" x2="10.16" y2="55.118" width="0" layer="20" curve="90"/>
-<wire x1="10.16" y1="55.118" x2="10.16" y2="12.5984" width="0" layer="20"/>
+<wire x1="10.16" y1="55.118" x2="10.16" y2="16.26" width="0" layer="20"/>
 <text x="59.182" y="36.322" size="0.8128" layer="21" rot="R90">MAC/PHY Ethernet Shield</text>
 <text x="59.182" y="50.038" size="0.8128" layer="21" rot="R90">v2.4</text>
+<wire x1="18.135" y1="15.725" x2="10.655" y2="15.725" width="0" layer="20"/>
+<wire x1="10.655" y1="15.725" x2="10.16" y2="16.22" width="0" layer="20" curve="-90"/>
+<wire x1="10.16" y1="16.22" x2="10.16" y2="16.26" width="0" layer="20"/>
 </plain>
 <attributes>
@@
 </class>
 </classes>
-<designrules name="default">
+<designrules>
 <description language="de">&lt;b&gt;EAGLE Design Rules&lt;/b&gt;
 &lt;p&gt;
