File: eagle/Camera Gantry Driver 1 - Axis/1-Axis Board - Camera Gantry.sch (EAGLE design)
At the start: 56 parts, among them U1 PTN78000, U2 DRV8312_DDW_44, U3 TPS61085_DGK_8

Commit message: More work on the new driver boards.
Parts:
- added JP5: M03SCREW_LOCK, ASL:M03SCREW_LOCK
- C1, C10, C2, C26, C27, C3, C5, C7: device CMPE118lib:CAP1206 -> ASL:CAP0805
- C19: device ASL:CAP1206 -> ASL:CAP0805
Connections:
- net OUT_A: now also JP5.3
- net OUT_B: now also JP5.2
- net OUT_C: now also JP5.1
Changed lines of the file:
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@@
 <?xml version="1.0" encoding="utf-8"?>
 <!DOCTYPE eagle SYSTEM "eagle.dtd">
-<eagle version="6.5.0">
+<eagle version="6.4">
 <drawing>
 <settings>
@@
 <layers>
 <layer number="1" name="Top" color="4" fill="1" visible="no" active="no"/>
+<layer number="2" name="Route2" color="1" fill="3" visible="no" active="no"/>
+<layer number="3" name="Route3" color="4" fill="3" visible="no" active="no"/>
+<layer number="4" name="Route4" color="1" fill="4" visible="no" active="no"/>
+<layer number="5" name="Route5" color="4" fill="4" visible="no" active="no"/>
+<layer number="6" name="Route6" color="1" fill="8" visible="no" active="no"/>
+<layer number="7" name="Route7" color="4" fill="8" visible="no" active="no"/>
+<layer number="8" name="Route8" color="1" fill="2" visible="no" active="no"/>
+<layer number="9" name="Route9" color="4" fill="2" visible="no" active="no"/>
+<layer number="10" name="Route10" color="1" fill="7" visible="no" active="no"/>
+<layer number="11" name="Route11" color="4" fill="7" visible="no" active="no"/>
+<layer number="12" name="Route12" color="1" fill="5" visible="no" active="no"/>
+<layer number="13" name="Route13" color="4" fill="5" visible="no" active="no"/>
+<layer number="14" name="Route14" color="1" fill="6" visible="no" active="no"/>
+<layer number="15" name="Route15" color="4" fill="6" visible="no" active="no"/>
 <layer number="16" name="Bottom" color="1" fill="1" visible="no" active="no"/>
 <layer number="17" name="Pads" color="2" fill="1" visible="no" active="no"/>
@@
 <part name="R1" library="CMPE118lib" deviceset="RESISTOR" device="0805-RES" value="330"/>
 <part name="GND7" library="CMPE118lib" deviceset="GND" device=""/>
-<part name="C7" library="CMPE118lib" deviceset="CAP" device="1206" value=".1uF"/>
+<part name="C7" library="ASL" deviceset="CAP" device="0805" value=".1uF"/>
 <part name="GND10" library="CMPE118lib" deviceset="GND" device=""/>
 <part name="R4" library="CMPE118lib" deviceset="RESISTOR" device="0805-RES" value="470"/>
@@
 <part name="GND11" library="CMPE118lib" deviceset="GND" device=""/>
 <part name="U$9" library="CMPE118lib" deviceset="VCC3V3" device=""/>
-<part name="C10" library="CMPE118lib" deviceset="CAP" device="1206" value=".1uF"/>
+<part name="C10" library="ASL" deviceset="CAP" device="0805" value=".1uF"/>
 <part name="LED2" library="CMPE118lib" deviceset="LED" device="1206">
 <attribute name="COLOR" value="red"/>
@@
 <part name="GND4" library="CMPE118lib" deviceset="GND" device=""/>
 <part name="C18" library="ASL" deviceset="CAP_POL" device="PTH4" value="1000uF"/>
-<part name="C19" library="ASL" deviceset="CAP" device="1206" value="10nF"/>
+<part name="C19" library="ASL" deviceset="CAP" device="0805" value="10nF"/>
 <part name="R10" library="ASL" deviceset="RESISTOR" device="0805-RES" value="3.3Ohm"/>
 <part name="GND9" library="ASL" deviceset="GND" device=""/>
 <part name="C6" library="ASL" deviceset="CAP_POL" device="PTH1" value="100uF"/>
 <part name="U$1" library="DRV83x2Support" deviceset="DSPIC33EP256MC506" device=""/>
-<part name="C1" library="CMPE118lib" deviceset="CAP" device="1206" value=".1uF"/>
-<part name="C2" library="CMPE118lib" deviceset="CAP" device="1206" value=".1uF"/>
-<part name="C3" library="CMPE118lib" deviceset="CAP" device="1206" value=".1uF"/>
-<part name="C5" library="CMPE118lib" deviceset="CAP" device="1206" value=".1uF"/>
+<part name="C1" library="ASL" deviceset="CAP" device="0805" value=".1uF"/>
+<part name="C2" library="ASL" deviceset="CAP" device="0805" value=".1uF"/>
+<part name="C3" library="ASL" deviceset="CAP" device="0805" value=".1uF"/>
+<part name="C5" library="ASL" deviceset="CAP" device="0805" value=".1uF"/>
 <part name="U2" library="DRV83x2Support" deviceset="DRV8312_DDW_44" device=""/>
 <part name="C8" library="ASL" deviceset="CAP" device="0805" value="1uF"/>
@@
 <part name="D5" library="DRV83x2Support" deviceset="PMEG2010AEH" device=""/>
 <part name="C25" library="ASL" deviceset="CAP" device="1206" value="10uF 16V"/>
-<part name="C26" library="CMPE118lib" deviceset="CAP" device="1206" value="1uF 16V"/>
-<part name="C27" library="CMPE118lib" deviceset="CAP" device="1206" value=".1uF"/>
+<part name="C26" library="ASL" deviceset="CAP" device="0805" value="1uF 16V"/>
+<part name="C27" library="ASL" deviceset="CAP" device="0805" value=".1uF"/>
 <part name="R9" library="ASL" deviceset="RESISTOR" device="0805-RES" value="18.2k"/>
 <part name="R11" library="ASL" deviceset="RESISTOR" device="0805-RES" value="158k"/>
@@
 <part name="SL1" library="ASL" deviceset="M04" device="LOCK"/>
 <part name="JP4" library="ASL" deviceset="M06" device="LOCK"/>
+<part name="JP5" library="ASL" deviceset="M03" device="SCREW_LOCK"/>
 </parts>
 <sheets>
@@
 <instance part="SL1" gate="G$1" x="139.7" y="38.1"/>
 <instance part="JP4" gate="G$1" x="383.54" y="-5.08" rot="R180"/>
+<instance part="JP5" gate="G$1" x="170.18" y="-58.42" rot="R270"/>
 </instances>
 <busses>
@@
 <wire x1="111.76" y1="-93.98" x2="111.76" y2="-96.52" width="0.1524" layer="91"/>
 </segment>
+<segment>
+<pinref part="JP5" gate="G$1" pin="1"/>
+<wire x1="172.72" y1="-66.04" x2="172.72" y2="-68.58" width="0.1524" layer="91"/>
+<label x="172.72" y="-73.66" size="1.778" layer="95" rot="R90"/>
+</segment>
 </net>
 <net name="N$30" class="0">
@@
 <wire x1="91.44" y1="-73.66" x2="111.76" y2="-73.66" width="0.1524" layer="91"/>
 </segment>
+<segment>
+<pinref part="JP5" gate="G$1" pin="2"/>
+<wire x1="170.18" y1="-66.04" x2="170.18" y2="-68.58" width="0.1524" layer="91"/>
+<label x="170.18" y="-73.66" size="1.778" layer="95" rot="R90"/>
+</segment>
 </net>
 <net name="OUT_A" class="0">
@@
 <wire x1="91.44" y1="-66.04" x2="111.76" y2="-66.04" width="0.1524" layer="91"/>
 </segment>
-</net>
+<segment>
+<pinref part="JP5" gate="G$1" pin="3"/>
+<wire x1="167.64" y1="-66.04" x2="167.64" y2="-68.58" width="0.1524" layer="91"/>
+<label x="167.64" y="-73.66" size="1.778" layer="95" rot="R90"/>
+</segment>
+</net>

Commit message: Did some clean-up to the directory, added an ams EasyPoint breakout board and consolidated PMSMmini board as well as pavlo.lbr.
Parts:
- removed JP2: (no value), ASL:M06LOCK
Connections:
- removed net N$17: JP2.1, U$1.RP118/RG6
- removed net N$19: JP2.4, U$1.FLT32/SCL2/RP36/RB4
- removed net N$20: JP2.5, U$1.PGED2/ASDA2/RP37/RB5
- removed net N$22: JP2.6, U$1.PGEC2/ASCL2/RP38/RB6
- removed net N$29: JP2.2, U$1.RP120/RG8
- removed net N$8: C1.1, U$1.AVDD
- removed net N$9: C1.2, U$1.AVSS
- net GND: now also C1.2, U$1.AVSS; no longer JP2.3
- net VCC: now also C1.1, U$1.AVDD
Other:
- moved on the sheet: U2
Changed lines of the file:
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@@
 <part name="C28" library="ASL" deviceset="CAP" device="1206" value="10uF"/>
 <part name="JP1" library="ASL" deviceset="M06" device="LOCK"/>
-<part name="JP2" library="ASL" deviceset="M06" device="LOCK"/>
 <part name="SL1" library="ASL" deviceset="M04" device="LOCK"/>
 <part name="JP4" library="ASL" deviceset="M06" device="LOCK"/>
@@
 <instance part="C28" gate="G$1" x="393.7" y="50.8" rot="R90"/>
 <instance part="JP1" gate="G$1" x="424.18" y="38.1" rot="R180"/>
-<instance part="JP2" gate="G$1" x="124.46" y="-2.54"/>
 <instance part="SL1" gate="G$1" x="139.7" y="38.1"/>
 <instance part="JP4" gate="G$1" x="383.54" y="-5.08" rot="R180"/>
@@
 </segment>
 <segment>
-<pinref part="JP2" gate="G$1" pin="3"/>
-<wire x1="134.62" y1="0" x2="129.54" y2="0" width="0.1524" layer="91"/>
-<label x="134.62" y="0" size="1.778" layer="95"/>
+<pinref part="U$1" gate="A" pin="AVSS"/>
+<wire x1="162.56" y1="22.86" x2="157.48" y2="22.86" width="0.1524" layer="91"/>
+<label x="152.4" y="22.86" size="1.778" layer="95"/>
+<wire x1="157.48" y1="22.86" x2="157.48" y2="20.32" width="0.1524" layer="91"/>
+<pinref part="C1" gate="G$1" pin="2"/>
+<wire x1="157.48" y1="20.32" x2="144.78" y2="20.32" width="0.1524" layer="91"/>
 </segment>
 </net>
@@
 <pinref part="C19" gate="G$1" pin="1"/>
 <pinref part="R10" gate="G$1" pin="1"/>
-</segment>
-</net>
-<net name="N$8" class="0">
-<segment>
-<pinref part="U$1" gate="A" pin="AVDD"/>
-<wire x1="162.56" y1="25.4" x2="157.48" y2="25.4" width="0.1524" layer="91"/>
-<label x="152.4" y="25.4" size="1.778" layer="95"/>
-<pinref part="C1" gate="G$1" pin="1"/>
-<wire x1="144.78" y1="27.94" x2="157.48" y2="27.94" width="0.1524" layer="91"/>
-<wire x1="157.48" y1="27.94" x2="157.48" y2="25.4" width="0.1524" layer="91"/>
-</segment>
-</net>
-<net name="N$9" class="0">
-<segment>
-<pinref part="U$1" gate="A" pin="AVSS"/>
-<wire x1="162.56" y1="22.86" x2="157.48" y2="22.86" width="0.1524" layer="91"/>
-<label x="152.4" y="22.86" size="1.778" layer="95"/>
-<wire x1="157.48" y1="22.86" x2="157.48" y2="20.32" width="0.1524" layer="91"/>
-<pinref part="C1" gate="G$1" pin="2"/>
-<wire x1="157.48" y1="20.32" x2="144.78" y2="20.32" width="0.1524" layer="91"/>
 </segment>
 </net>
@@
 <wire x1="220.98" y1="-78.74" x2="218.44" y2="-78.74" width="0.1524" layer="91"/>
 <label x="213.36" y="-78.74" size="1.778" layer="95"/>
+</segment>
+<segment>
+<pinref part="U$1" gate="A" pin="AVDD"/>
+<wire x1="162.56" y1="25.4" x2="157.48" y2="25.4" width="0.1524" layer="91"/>
+<label x="152.4" y="25.4" size="1.778" layer="95"/>
+<pinref part="C1" gate="G$1" pin="1"/>
+<wire x1="144.78" y1="27.94" x2="157.48" y2="27.94" width="0.1524" layer="91"/>
+<wire x1="157.48" y1="27.94" x2="157.48" y2="25.4" width="0.1524" layer="91"/>
 </segment>
 </net>
@@
 </segment>
 </net>
-<net name="N$17" class="0">
-<segment>
-<pinref part="U$1" gate="A" pin="RP118/RG6"/>
-<pinref part="JP2" gate="G$1" pin="1"/>
-<wire x1="162.56" y1="63.5" x2="129.54" y2="63.5" width="0.1524" layer="91"/>
-<wire x1="129.54" y1="63.5" x2="129.54" y2="5.08" width="0.1524" layer="91"/>
-</segment>
-</net>
-<net name="N$19" class="0">
-<segment>
-<pinref part="U$1" gate="A" pin="FLT32/SCL2/RP36/RB4"/>
-<wire x1="162.56" y1="-7.62" x2="137.16" y2="-7.62" width="0.1524" layer="91"/>
-<wire x1="137.16" y1="-7.62" x2="137.16" y2="-2.54" width="0.1524" layer="91"/>
-<pinref part="JP2" gate="G$1" pin="4"/>
-<wire x1="137.16" y1="-2.54" x2="129.54" y2="-2.54" width="0.1524" layer="91"/>
-</segment>
-</net>
-<net name="N$20" class="0">
-<segment>
-<pinref part="U$1" gate="A" pin="PGED2/ASDA2/RP37/RB5"/>
-<wire x1="365.76" y1="17.78" x2="398.78" y2="17.78" width="0.1524" layer="91"/>
-<wire x1="398.78" y1="17.78" x2="398.78" y2="-25.4" width="0.1524" layer="91"/>
-<wire x1="398.78" y1="-25.4" x2="134.62" y2="-25.4" width="0.1524" layer="91"/>
-<wire x1="134.62" y1="-25.4" x2="134.62" y2="-5.08" width="0.1524" layer="91"/>
-<pinref part="JP2" gate="G$1" pin="5"/>
-<wire x1="134.62" y1="-5.08" x2="129.54" y2="-5.08" width="0.1524" layer="91"/>
-</segment>
-</net>
-<net name="N$22" class="0">
-<segment>
-<pinref part="U$1" gate="A" pin="PGEC2/ASCL2/RP38/RB6"/>
-<wire x1="365.76" y1="20.32" x2="403.86" y2="20.32" width="0.1524" layer="91"/>
-<wire x1="403.86" y1="20.32" x2="403.86" y2="-30.48" width="0.1524" layer="91"/>
-<pinref part="JP2" gate="G$1" pin="6"/>
-<wire x1="403.86" y1="-30.48" x2="129.54" y2="-30.48" width="0.1524" layer="91"/>
-<wire x1="129.54" y1="-30.48" x2="129.54" y2="-7.62" width="0.1524" layer="91"/>
-</segment>
-</net>
 <net name="N$23" class="0">
 <segment>
@@
 </segment>
 </net>
-<net name="N$29" class="0">
-<segment>
-<pinref part="U$1" gate="A" pin="RP120/RG8"/>
-<pinref part="JP2" gate="G$1" pin="2"/>
-<wire x1="129.54" y1="2.54" x2="132.08" y2="2.54" width="0.1524" layer="91"/>
-<wire x1="132.08" y1="2.54" x2="132.08" y2="58.42" width="0.1524" layer="91"/>
-<wire x1="132.08" y1="58.42" x2="162.56" y2="58.42" width="0.1524" layer="91"/>
-</segment>
-</net>
