File: eagle/CMPE121 Final Project/LED Matrix/MatrixDriver.brd (EAGLE design)
At the start: 100 x 80 mm, 25 parts, among them J1 M16DUAL_ROW, J2 M16DUAL_ROW

Commit message: Finished gerbers.
Parts:
- moved R1 11.2 mm to (70.1, 38.9)
- moved R2 11.2 mm to (70.1, 33.8)
- moved R3 11.2 mm to (70.1, 28.7)
- moved R4 11.2 mm to (70.1, 23.6)
- moved RN5 1.27 mm to (41.9, 70.9)
- moved RN6 1.27 mm to (36.8, 70.9)
- moved J2 1.27 mm to (35.6, 76.2)
Routing:
- net VDD5V0: track 0.00 -> 202.2 mm, vias 0 -> 1
- net N$9: track 0.00 -> 93.4 mm, vias 0 -> 2
- net N$11: track 0.00 -> 90.4 mm, vias 0 -> 2
- net N$60: track 0.00 -> 84.2 mm
- net N$59: track 0.00 -> 81.1 mm
- net N$61: track 0.00 -> 77.6 mm, vias 0 -> 2
- net N$58: track 0.00 -> 72.5 mm
- net N$57: track 0.00 -> 69.3 mm
- net N$62: track 0.00 -> 68.5 mm, vias 0 -> 2
- net N$63: track 0.00 -> 63.3 mm
- net N$10: track 0.00 -> 60.5 mm, vias 0 -> 2
- net N$12: track 0.00 -> 58.0 mm, vias 0 -> 2
- net N$64: track 0.00 -> 54.8 mm
- net ROW2: track 0.00 -> 8.24 mm
- net ROW1: track 0.00 -> 8.21 mm
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Other:
- board size 100 x 80 mm -> 81.2 x 80 mm
