File: eagle/Nanopore Amp/CurrentAmp.brd (EAGLE design)
At the start: 53 x 62 mm, 27 parts, among them IC1 AD820RM, IC2 AD820RM, IC3 OPA129U, X1 1-227161-0, X2 1-227161-0, X3 1-227161-0, X4 1-227161-0, X5 1-227161-0, X6 1-227161-0

Commit message: Current amp work.
Parts:
- removed X2: 1-227161-0, con-coax:AMP_227161
- added JP1: M03PTH, ASL:1X03
- moved C3 16.1 mm to (26.2, 33.7)
- moved C4 16.1 mm to (20.2, 28.4)
- moved R3 16.1 mm to (23.2, 26.5)
- moved R4 16.1 mm to (25.0, 26.5)
- moved IC2 16.1 mm to (24.0, 30.5)
- moved X6 16.1 mm to (8.00, 31.1)
- moved R7 16.0 mm to (16.5, 27.6)
- moved X5 15.3 mm to (42.0, 15.8)
- moved C5 15.1 mm to (20.9, 19.0)
- moved C6 15.1 mm to (23.2, 11.0)
- moved IC3 15.1 mm to (24.0, 15.0)
- moved R5 15.1 mm to (23.9, 18.5)
- moved R8 15.0 mm to (16.0, 12.0)
- moved X3 15.0 mm to (8.00, 15.8)
- moved E$2 3.00 mm to (46.0, 4.00)
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Connections:
- removed net N$2: IC1.6, R1.2, X4.1
- net GND: now also IC3.8, JP1.2; no longer X2.2
- net HVDD_15: now also JP1.1
- net HVSS_15: now also JP1.3
- net N$6: now also IC1.6, R1.2, X4.1; no longer X2.1
Routing:
- net N$10: track 0.00 -> 28.4 mm
- net N$6: track 17.6 -> 39.7 mm
- net N$2: track 15.9 -> 0.00 mm
- net GND: track 0.00 -> 7.07 mm, vias 200 -> 193
- net HVDD_15: track 60.2 -> 66.1 mm
- net HVSS_15: track 49.8 -> 55.4 mm, vias 3 -> 4
- net N$3: track 10.7 -> 8.70 mm
- net N$7: track 15.0 -> 13.0 mm
- net N$5: track 15.4 -> 13.4 mm
- net N$8: track 16.3 -> 15.3 mm
Other:
- board size 53 x 62 mm -> 50 x 62 mm
- board text added: "+15V"
- board text added: "-15V"
- board text added: "GND"
- board text added: "Nanopore Current Amp Pavlo Manovi - (c) 2014 http://pavlo.me"
- board text added: "Released under the TAPR OHL."

Commit message: Fixed current amp board.
Connections:
- net GND: now also IC2.3, IC3.3; no longer IC2.2, IC3.2
- net N$4: now also IC2.2; no longer IC2.3
- net N$8: now also IC3.2; no longer IC3.3
Routing:
- net N$8: track 15.3 -> 17.6 mm
- net N$4: track 7.05 -> 6.54 mm
- net GND: vias 193 -> 192
Other:
- board text added: "Nanopore Current Amp v1.1 Pavlo Manovi - (c) 2014 http://pavlo.me"
- board text removed: "Nanopore Current Amp Pavlo Manovi - (c) 2014 http://pavlo.me"
Changed lines of the file:
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@@
 <text x="35.1" y="23" size="1.27" layer="25" font="vector" rot="R180">From
 Membrane</text>
-<text x="23.1" y="60.4" size="1.016" layer="25" rot="R180">+15V</text>
+<text x="27.9" y="60.6" size="1.016" layer="25" rot="R180">+15V</text>
 <text x="23.7" y="53.5" size="1.016" layer="25" rot="R90">GND</text>
-<text x="25" y="59.4" size="1.016" layer="25">-15V</text>
+<text x="19.8" y="59.6" size="1.016" layer="25">-15V</text>
 <polygon width="0.2" layer="22">
 <vertex x="11.610715625" y="54.6945" curve="-9.499997"/>
@@
 </polygon>
 <text x="41.3" y="54.8" size="1.016" layer="26" rot="MR0">Released under the TAPR OHL.</text>
-<text x="41.1" y="3" size="1.016" layer="26" rot="MR0">Nanopore Current Amp
+<text x="41.1" y="3" size="1.016" layer="26" rot="MR0">Nanopore Current Amp v1.1
 Pavlo Manovi - (c) 2014
 http://pavlo.me</text>
@@
 </signal>
 <signal name="N$4">
-<contactref element="IC2" pad="3"/>
+<contactref element="R3" pad="2"/>
 <contactref element="R4" pad="1"/>
-<contactref element="R3" pad="2"/>
-<wire x1="26.263" y1="30.82" x2="25.52" y2="30.82" width="0.4064" layer="1"/>
-<wire x1="25.52" y1="30.82" x2="24.9" y2="30.2" width="0.4064" layer="1"/>
-<wire x1="24.9" y1="30.2" x2="24.9" y2="27.5" width="0.4064" layer="1"/>
-<wire x1="24.9" y1="27.5" x2="25" y2="27.4" width="0.4064" layer="1"/>
-<wire x1="23.156" y1="25.6" x2="23.2" y2="25.6" width="0.4064" layer="1"/>
-<wire x1="23.2" y1="25.6" x2="25" y2="27.4" width="0.4064" layer="1"/>
+<contactref element="IC2" pad="2"/>
+<wire x1="25" y1="27.4" x2="24.956" y2="27.4" width="0.4064" layer="1"/>
+<wire x1="24.956" y1="27.4" x2="24.628" y2="27.072" width="0.4064" layer="1"/>
+<wire x1="24.628" y1="27.072" x2="23.156" y2="25.6" width="0.4064" layer="1"/>
+<wire x1="26.263" y1="30.17" x2="25.17" y2="30.17" width="0.4064" layer="1"/>
+<wire x1="25.17" y1="30.17" x2="25" y2="30" width="0.4064" layer="1"/>
+<wire x1="25" y1="30" x2="25" y2="27.444" width="0.4064" layer="1"/>
+<wire x1="25" y1="27.444" x2="24.956" y2="27.4" width="0.4064" layer="1"/>
 </signal>
 <signal name="N$5">
@@
 </signal>
 <signal name="N$8">
-<contactref element="X5" pad="1"/>
-<contactref element="IC3" pad="3"/>
 <contactref element="R5" pad="2"/>
-<wire x1="26.6162" y1="15.617" x2="24.883" y2="15.617" width="0.4064" layer="1"/>
 <wire x1="24.883" y1="15.617" x2="24.6" y2="15.9" width="0.4064" layer="1"/>
 <wire x1="24.6" y1="15.9" x2="24.6" y2="18.528" width="0.4064" layer="1"/>
 <wire x1="24.6" y1="18.528" x2="24.81" y2="18.538" width="0.4064" layer="1"/>
-<wire x1="26.6162" y1="15.617" x2="36.737" y2="15.617" width="0.4064" layer="1"/>
-<wire x1="36.737" y1="15.617" x2="36.92" y2="15.75" width="0.4064" layer="1"/>
+<contactref element="X5" pad="1"/>
+<contactref element="IC3" pad="2"/>
+<wire x1="26.6162" y1="14.347" x2="36.347" y2="14.347" width="0.4064" layer="1"/>
+<wire x1="36.347" y1="14.347" x2="36.9" y2="14.9" width="0.4064" layer="1"/>
+<wire x1="36.9" y1="14.9" x2="36.9" y2="15.73" width="0.4064" layer="1"/>
+<wire x1="36.9" y1="15.73" x2="36.92" y2="15.75" width="0.4064" layer="1"/>
+<wire x1="24.883" y1="15.617" x2="24.883" y2="14.417" width="0.4064" layer="1"/>
+<wire x1="24.883" y1="14.417" x2="25" y2="14.3" width="0.4064" layer="1"/>
+<wire x1="25" y1="14.3" x2="26.5692" y2="14.3" width="0.4064" layer="1"/>
+<wire x1="26.5692" y1="14.3" x2="26.6162" y2="14.347" width="0.4064" layer="1"/>
 </signal>
 <signal name="GND">
 <contactref element="R2" pad="1"/>
-<contactref element="IC3" pad="2"/>
-<contactref element="IC2" pad="2"/>
 <contactref element="C1" pad="2"/>
 <contactref element="C2" pad="2"/>
@@
 <via x="17.5" y="14.5" extent="1-16" drill="0.4" shape="square"/>
 <via x="18.5" y="14.5" extent="1-16" drill="0.4" shape="square"/>
-<via x="29.5" y="16.8" extent="1-16" drill="0.4" shape="square"/>
-<via x="30.5" y="16.8" extent="1-16" drill="0.4" shape="square"/>
-<via x="31.5" y="16.8" extent="1-16" drill="0.4" shape="square"/>
-<via x="32.5" y="16.8" extent="1-16" drill="0.4" shape="square"/>
-<via x="33.5" y="16.8" extent="1-16" drill="0.4" shape="square"/>
-<via x="34.5" y="16.8" extent="1-16" drill="0.4" shape="square"/>
-<via x="35.5" y="16.8" extent="1-16" drill="0.4" shape="square"/>
-<via x="29.5" y="14.5" extent="1-16" drill="0.4" shape="square"/>
-<via x="30.5" y="14.5" extent="1-16" drill="0.4" shape="square"/>
-<via x="31.5" y="14.5" extent="1-16" drill="0.4" shape="square"/>
-<via x="32.5" y="14.5" extent="1-16" drill="0.4" shape="square"/>
-<via x="33.5" y="14.5" extent="1-16" drill="0.4" shape="square"/>
-<via x="34.5" y="14.5" extent="1-16" drill="0.4" shape="square"/>
-<via x="35.5" y="14.5" extent="1-16" drill="0.4" shape="square"/>
+<via x="28.7" y="15.3" extent="1-16" drill="0.4" shape="square"/>
+<via x="29.7" y="15.3" extent="1-16" drill="0.4" shape="square"/>
+<via x="30.7" y="15.3" extent="1-16" drill="0.4" shape="square"/>
+<via x="31.7" y="15.3" extent="1-16" drill="0.4" shape="square"/>
+<via x="32.7" y="15.3" extent="1-16" drill="0.4" shape="square"/>
+<via x="33.7" y="15.3" extent="1-16" drill="0.4" shape="square"/>
+<via x="34.7" y="15.3" extent="1-16" drill="0.4" shape="square"/>
+<via x="29.7" y="13" extent="1-16" drill="0.4" shape="square"/>
+<via x="30.7" y="13" extent="1-16" drill="0.4" shape="square"/>
+<via x="31.7" y="13" extent="1-16" drill="0.4" shape="square"/>
+<via x="32.7" y="13" extent="1-16" drill="0.4" shape="square"/>
+<via x="33.7" y="13" extent="1-16" drill="0.4" shape="square"/>
+<via x="34.7" y="13" extent="1-16" drill="0.4" shape="square"/>
 <via x="1.5" y="54.5" extent="1-16" drill="0.4" shape="square"/>
 <via x="1.5" y="52.5" extent="1-16" drill="0.4" shape="square"/>
@@
 <wire x1="28.5" y1="17.5" x2="28.6" y2="17.6" width="0.4064" layer="1"/>
 <wire x1="25.6" y1="13.1" x2="24.9" y2="13.8" width="0.4064" layer="1"/>
-<via x="24" y="15" extent="1-16" drill="0.4" shape="octagon"/>
+<via x="23.8" y="15" extent="1-16" drill="0.4" shape="octagon"/>
 <via x="23.9" y="19.9" extent="1-16" drill="0.4" shape="octagon"/>
 <via x="28.3" y="18" extent="1-16" drill="0.4" shape="octagon"/>
@@
 <via x="41.5" y="1.5" extent="1-16" drill="0.4" shape="square"/>
 <via x="1.5" y="7.5" extent="1-16" drill="0.4" shape="square"/>
+<contactref element="IC3" pad="3"/>
+<contactref element="IC2" pad="3"/>
 </signal>
 <signal name="HVDD_15">
