File: eagle/Nanopore Amp/CurrentAmp.sch (EAGLE design)
At the start: 23 parts, among them IC1 AD820RM, IC2 AD820RM, IC3 OPA129U, X1 1-227161-0, X2 1-227161-0, X3 1-227161-0, X4 1-227161-0, X5 1-227161-0, X6 1-227161-0

Commit message: Current amp work.
Parts:
- removed X2: 1-227161-0, con-coax:1-227161-0
- added JP1: M03PTH, ASL:M03PTH
Connections:
- removed net N$2: IC1.OUT, R1.2, X4.1
- net GND: now also IC3.SUBS, JP1.2; no longer X2.2
- net HVDD_15: now also JP1.1
- net HVSS_15: now also JP1.3
- net N$6: now also IC1.OUT, R1.2, X4.1; no longer X2.1
Changed lines of the file:
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@@
 <layer number="203" name="203bmp" color="4" fill="10" visible="no" active="yes"/>
 <layer number="204" name="204bmp" color="5" fill="10" visible="no" active="yes"/>
-<layer number="205" name="205bmp" color="6" fill="10" visible="no" active="yes"/>
+<layer number="205" name="205bmp" color="6" fill="10" visible="yes" active="yes"/>
 <layer number="206" name="206bmp" color="7" fill="10" visible="yes" active="yes"/>
 <layer number="207" name="207bmp" color="8" fill="10" visible="no" active="yes"/>
@@
 <part name="IC3" library="burr-brown" deviceset="OPA129" device="U"/>
 <part name="X1" library="con-coax" deviceset="?227161*" device="1-" technology="-0"/>
-<part name="X2" library="con-coax" deviceset="?227161*" device="1-" technology="-0"/>
 <part name="X3" library="con-coax" deviceset="?227161*" device="1-" technology="-0"/>
 <part name="R1" library="ASL" deviceset="RESISTOR" device="0805-RES" value="5M 1%"/>
@@
 <part name="R7" library="ASL" deviceset="RESISTOR" device="0805-RES" value="10k"/>
 <part name="R8" library="ASL" deviceset="RESISTOR" device="0805-RES" value="10k"/>
+<part name="JP1" library="ASL" deviceset="M03" device="PTH"/>
 </parts>
 <sheets>
 <sheet>
 <plain>
-<rectangle x1="88.9" y1="12.7" x2="147.32" y2="88.9" layer="206"/>
 <text x="106.68" y="88.9" size="1.778" layer="206">Nanopore/Membrane</text>
 <wire x1="91.44" y1="71.12" x2="101.6" y2="71.12" width="0.1524" layer="94"/>
@@
 <wire x1="116.84" y1="83.82" x2="132.08" y2="83.82" width="0.1524" layer="94"/>
 <wire x1="132.08" y1="83.82" x2="132.08" y2="71.12" width="0.1524" layer="94"/>
-<wire x1="144.78" y1="38.1" x2="101.6" y2="38.1" width="0.1524" layer="94"/>
-<wire x1="101.6" y1="38.1" x2="101.6" y2="71.12" width="0.1524" layer="94"/>
 <circle x="101.6" y="71.12" radius="0.567959375" width="0.1524" layer="94"/>
 <circle x="132.08" y="71.12" radius="0.567959375" width="0.1524" layer="94"/>
 <circle x="144.78" y="71.12" radius="0.508" width="0.1524" layer="94"/>
 <circle x="91.44" y="71.12" radius="0.508" width="0.1524" layer="94"/>
-<circle x="144.78" y="38.1" radius="0.508" width="0.1524" layer="94"/>
+<rectangle x1="88.9" y1="55.88" x2="147.32" y2="88.9" layer="205"/>
 </plain>
 <instances>
@@
 <instance part="IC3" gate="G$1" x="180.34" y="71.12"/>
 <instance part="X1" gate="G$1" x="12.7" y="73.66"/>
-<instance part="X2" gate="G$1" x="152.4" y="38.1"/>
 <instance part="X3" gate="G$1" x="223.52" y="71.12" rot="MR0"/>
 <instance part="R1" gate="G$1" x="68.58" y="63.5" rot="R90"/>
@@
 <instance part="R7" gate="G$1" x="213.36" y="33.02"/>
 <instance part="R8" gate="G$1" x="213.36" y="68.58"/>
+<instance part="JP1" gate="G$1" x="17.78" y="30.48" rot="R270"/>
 </instances>
 <busses>
@@
 <junction x="68.58" y="55.88"/>
 <wire x1="68.58" y1="55.88" x2="68.58" y2="58.42" width="0.1524" layer="91"/>
-</segment>
-</net>
-<net name="N$2" class="0">
-<segment>
-<pinref part="IC1" gate="G$1" pin="OUT"/>
-<wire x1="53.34" y1="71.12" x2="68.58" y2="71.12" width="0.1524" layer="91"/>
-<pinref part="R1" gate="G$1" pin="2"/>
-<wire x1="68.58" y1="68.58" x2="68.58" y2="71.12" width="0.1524" layer="91"/>
-<junction x="68.58" y="71.12"/>
-<pinref part="X4" gate="G$1" pin="1"/>
-<wire x1="81.28" y1="71.12" x2="68.58" y2="71.12" width="0.1524" layer="91"/>
 </segment>
 </net>
@@
 <wire x1="185.42" y1="81.28" x2="187.96" y2="81.28" width="0.1524" layer="91"/>
 <label x="187.96" y="81.28" size="1.778" layer="95"/>
+<pinref part="IC3" gate="G$1" pin="SUBS"/>
+<wire x1="187.96" y1="73.66" x2="187.96" y2="81.28" width="0.1524" layer="91"/>
 </segment>
 <segment>
@@
 </segment>
 <segment>
-<pinref part="X2" gate="G$1" pin="2"/>
-<wire x1="154.94" y1="35.56" x2="157.48" y2="35.56" width="0.1524" layer="91"/>
-<label x="157.48" y="35.56" size="1.778" layer="95"/>
+<pinref part="JP1" gate="G$1" pin="2"/>
+<wire x1="17.78" y1="22.86" x2="17.78" y2="17.78" width="0.1524" layer="91"/>
+<wire x1="17.78" y1="17.78" x2="22.86" y2="17.78" width="0.1524" layer="91"/>
+<label x="22.86" y="17.78" size="1.778" layer="95"/>
 </segment>
 </net>
@@
 <junction x="180.34" y="43.18"/>
 </segment>
+<segment>
+<pinref part="JP1" gate="G$1" pin="1"/>
+<wire x1="20.32" y1="22.86" x2="20.32" y2="20.32" width="0.1524" layer="91"/>
+<wire x1="20.32" y1="20.32" x2="22.86" y2="20.32" width="0.1524" layer="91"/>
+<label x="22.86" y="20.32" size="1.778" layer="95"/>
+</segment>
 </net>
 <net name="HVSS_15" class="0">
@@
 <junction x="180.34" y="27.94"/>
 </segment>
+<segment>
+<pinref part="JP1" gate="G$1" pin="3"/>
+<wire x1="15.24" y1="22.86" x2="15.24" y2="15.24" width="0.1524" layer="91"/>
+<wire x1="15.24" y1="15.24" x2="22.86" y2="15.24" width="0.1524" layer="91"/>
+<label x="22.86" y="15.24" size="1.778" layer="95"/>
+</segment>
 </net>
 <net name="N$6" class="0">
 <segment>
 <pinref part="R4" gate="G$1" pin="2"/>
-<pinref part="X2" gate="G$1" pin="1"/>
-<wire x1="157.48" y1="38.1" x2="154.94" y2="38.1" width="0.1524" layer="91"/>
-</segment>
-</net>
+<pinref part="IC1" gate="G$1" pin="OUT"/>
+<wire x1="53.34" y1="71.12" x2="68.58" y2="71.12" width="0.1524" layer="91"/>
+<pinref part="R1" gate="G$1" pin="2"/>
+<wire x1="68.58" y1="68.58" x2="68.58" y2="71.12" width="0.1524" layer="91"/>
+<junction x="68.58" y="71.12"/>
+<pinref part="X4" gate="G$1" pin="1"/>
+<wire x1="81.28" y1="71.12" x2="73.66" y2="71.12" width="0.1524" layer="91"/>
+<wire x1="73.66" y1="71.12" x2="68.58" y2="71.12" width="0.1524" layer="91"/>
+<wire x1="157.48" y1="38.1" x2="73.66" y2="38.1" width="0.1524" layer="91"/>
+<wire x1="73.66" y1="38.1" x2="73.66" y2="71.12" width="0.1524" layer="91"/>
+<junction x="73.66" y="71.12"/>
+</segment>
+</net>

Commit message: Fixed current amp board.
Connections:
- net GND: now also IC2.IN+, IC3.+IN; no longer IC2.IN-, IC3.-IN
- net N$4: now also IC2.IN-; no longer IC2.IN+
- net N$8: now also IC3.-IN; no longer IC3.+IN
Changed lines of the file:
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@@
 <net name="N$4" class="0">
 <segment>
-<pinref part="IC2" gate="G$1" pin="IN+"/>
+<pinref part="R3" gate="G$1" pin="2"/>
+<wire x1="183.134" y1="50.8" x2="167.64" y2="50.8" width="0.1524" layer="91"/>
 <pinref part="R4" gate="G$1" pin="1"/>
-<wire x1="172.72" y1="38.1" x2="167.64" y2="38.1" width="0.1524" layer="91"/>
-<pinref part="R3" gate="G$1" pin="2"/>
-<wire x1="183.134" y1="50.8" x2="172.72" y2="50.8" width="0.1524" layer="91"/>
-<wire x1="172.72" y1="50.8" x2="172.72" y2="38.1" width="0.1524" layer="91"/>
-<junction x="172.72" y="38.1"/>
+<wire x1="167.64" y1="50.8" x2="167.64" y2="38.1" width="0.1524" layer="91"/>
+<wire x1="167.64" y1="38.1" x2="167.64" y2="33.02" width="0.1524" layer="91"/>
+<pinref part="IC2" gate="G$1" pin="IN-"/>
+<wire x1="167.64" y1="33.02" x2="172.72" y2="33.02" width="0.1524" layer="91"/>
+<junction x="167.64" y="38.1"/>
 </segment>
 </net>
@@
 <net name="N$8" class="0">
 <segment>
+<pinref part="R5" gate="G$1" pin="2"/>
+<wire x1="180.34" y1="88.9" x2="170.18" y2="88.9" width="0.1524" layer="91"/>
+<wire x1="170.18" y1="88.9" x2="170.18" y2="71.12" width="0.1524" layer="91"/>
 <pinref part="X5" gate="G$1" pin="1"/>
-<wire x1="154.94" y1="71.12" x2="162.56" y2="71.12" width="0.1524" layer="91"/>
-<wire x1="162.56" y1="71.12" x2="162.56" y2="73.66" width="0.1524" layer="91"/>
-<pinref part="IC3" gate="G$1" pin="+IN"/>
-<wire x1="162.56" y1="73.66" x2="170.18" y2="73.66" width="0.1524" layer="91"/>
-<pinref part="R5" gate="G$1" pin="2"/>
-<wire x1="170.18" y1="73.66" x2="172.72" y2="73.66" width="0.1524" layer="91"/>
-<wire x1="180.34" y1="88.9" x2="170.18" y2="88.9" width="0.1524" layer="91"/>
-<wire x1="170.18" y1="88.9" x2="170.18" y2="73.66" width="0.1524" layer="91"/>
+<pinref part="IC3" gate="G$1" pin="-IN"/>
+<wire x1="154.94" y1="71.12" x2="170.18" y2="71.12" width="0.1524" layer="91"/>
+<wire x1="170.18" y1="71.12" x2="170.18" y2="68.58" width="0.1524" layer="91"/>
+<wire x1="170.18" y1="68.58" x2="172.72" y2="68.58" width="0.1524" layer="91"/>
+<junction x="170.18" y="71.12"/>
 </segment>
 </net>
@@
 </segment>
 <segment>
-<pinref part="IC3" gate="G$1" pin="-IN"/>
-<wire x1="172.72" y1="68.58" x2="167.64" y2="68.58" width="0.1524" layer="91"/>
-<wire x1="167.64" y1="68.58" x2="167.64" y2="58.42" width="0.1524" layer="91"/>
+<wire x1="167.64" y1="73.66" x2="167.64" y2="58.42" width="0.1524" layer="91"/>
 <label x="165.1" y="55.88" size="1.778" layer="95"/>
+<pinref part="IC3" gate="G$1" pin="+IN"/>
+<wire x1="167.64" y1="73.66" x2="172.72" y2="73.66" width="0.1524" layer="91"/>
 </segment>
 <segment>
-<pinref part="IC2" gate="G$1" pin="IN-"/>
-<wire x1="172.72" y1="33.02" x2="167.64" y2="33.02" width="0.1524" layer="91"/>
-<wire x1="167.64" y1="33.02" x2="167.64" y2="25.4" width="0.1524" layer="91"/>
-<label x="165.1" y="22.86" size="1.778" layer="95"/>
+<wire x1="170.18" y1="38.1" x2="170.18" y2="25.4" width="0.1524" layer="91"/>
+<label x="167.64" y="22.86" size="1.778" layer="95"/>
+<pinref part="IC2" gate="G$1" pin="IN+"/>
+<wire x1="172.72" y1="38.1" x2="170.18" y2="38.1" width="0.1524" layer="91"/>
 </segment>
 <segment>
